File: pcb/base_board/rev 1/baseboard.brd (EAGLE design)
At the start: 88 x 85 mm, 38 parts, among them IC1 LD117AS33TR, SW1 324_SW, SW2 324_SW, SW20 324_SW, SW3 324_SW, SW4 324_SW, U5 CH340C

Commit message: updated PCBs
Parts:
- removed JP6: (no value), pinhead:2X03
- added JP3, JP4: (no value), pinhead:1X03
- moved R5 9.65 mm to (79.4, 62.2)
- moved SW2 9.65 mm to (78.1, 72.4)
- moved SW3 9.65 mm to (78.1, 65.8)
- moved C20 0.92 mm to (2.20, 28.7)
Connections:
- net +3V3: now also JP3.1, JP3.2, JP3.3; no longer JP6.2, JP6.4, JP6.6
- net GND: now also JP4.1, JP4.2, JP4.3; no longer JP6.1, JP6.3, JP6.5
Routing:
- net N$6: track 103.3 -> 93.7 mm
- net N$32: track 38.4 -> 28.7 mm
- net GND: track 32.7 -> 26.2 mm
- net N$35: track 3.09 -> 2.33 mm
- net N$36: track 4.93 -> 4.18 mm
Other:
- outline, holes or cut-outs redrawn
- board text added: "G"
- board text removed: "GND"
