File: pcb/base_board/rev 1/baseboard.sch (EAGLE design)
At the start: 38 parts, among them IC1 LD117AS33TR, SW1 324_SW, SW2 324_SW, SW20 324_SW, SW3 324_SW, SW4 324_SW, U5 CH340C

Commit message: updated PCBs
Parts:
- removed JP6: (no value), pinhead:PINHD-2X3
- added JP3, JP4: (no value), pinhead:PINHD-1X3
Connections:
- net +3V3: now also JP3.1, JP3.2, JP3.3; no longer JP6.2, JP6.4, JP6.6
- net GND: now also JP4.1, JP4.2, JP4.3; no longer JP6.1, JP6.3, JP6.5
Changed lines of the file:
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@@
 <part name="+3V1" library="supply1" library_urn="urn:adsk.eagle:library:371" deviceset="+3V3" device=""/>
 <part name="+3V4" library="supply1" library_urn="urn:adsk.eagle:library:371" deviceset="+3V3" device=""/>
+<part name="JP3" library="pinhead" library_urn="urn:adsk.eagle:library:325" deviceset="PINHD-1X3" device="" package3d_urn="urn:adsk.eagle:package:22458/2"/>
+<part name="JP4" library="pinhead" library_urn="urn:adsk.eagle:library:325" deviceset="PINHD-1X3" device="" package3d_urn="urn:adsk.eagle:package:22458/2"/>
 <part name="JP5" library="pinhead" library_urn="urn:adsk.eagle:library:325" deviceset="PINHD-1X3" device="" package3d_urn="urn:adsk.eagle:package:22458/2"/>
 <part name="P+3" library="supply1" library_urn="urn:adsk.eagle:library:371" deviceset="+5V" device=""/>
@@
 <part name="+3V13" library="supply1" library_urn="urn:adsk.eagle:library:371" deviceset="+3V3" device=""/>
 <part name="+3V15" library="supply1" library_urn="urn:adsk.eagle:library:371" deviceset="+3V3" device=""/>
-<part name="JP6" library="pinhead" library_urn="urn:adsk.eagle:library:325" deviceset="PINHD-2X3" device="" package3d_urn="urn:adsk.eagle:package:22462/2"/>
 </parts>
 <sheets>
@@
 <attribute name="VALUE" x="480.06" y="50.8" size="1.778" layer="96" rot="R90"/>
 </instance>
+<instance part="JP3" gate="A" x="802.64" y="109.22" smashed="yes">
+<attribute name="NAME" x="796.29" y="114.935" size="1.778" layer="95"/>
+<attribute name="VALUE" x="796.29" y="101.6" size="1.778" layer="96"/>
+</instance>
+<instance part="JP4" gate="A" x="802.64" y="91.44" smashed="yes">
+<attribute name="NAME" x="796.29" y="97.155" size="1.778" layer="95"/>
+<attribute name="VALUE" x="796.29" y="83.82" size="1.778" layer="96"/>
+</instance>
 <instance part="JP5" gate="A" x="802.64" y="71.12" smashed="yes">
 <attribute name="NAME" x="796.29" y="76.835" size="1.778" layer="95"/>
@@
 <attribute name="VALUE" x="815.34" y="71.12" size="1.778" layer="96" rot="MR90"/>
 </instance>
-<instance part="+3V6" gate="G$1" x="772.16" y="111.76" smashed="yes">
-<attribute name="VALUE" x="769.62" y="106.68" size="1.778" layer="96" rot="R90"/>
-</instance>
-<instance part="GND4" gate="1" x="764.54" y="86.36" smashed="yes">
-<attribute name="VALUE" x="762" y="83.82" size="1.778" layer="96"/>
+<instance part="+3V6" gate="G$1" x="812.8" y="114.3" smashed="yes">
+<attribute name="VALUE" x="810.26" y="109.22" size="1.778" layer="96" rot="R90"/>
+</instance>
+<instance part="GND4" gate="1" x="810.26" y="86.36" smashed="yes">
+<attribute name="VALUE" x="807.72" y="83.82" size="1.778" layer="96"/>
 </instance>
 <instance part="SW2" gate="G$1" x="495.3" y="124.46" smashed="yes" rot="MR90"/>
@@
 <instance part="+3V15" gate="G$1" x="716.28" y="55.88" smashed="yes">
 <attribute name="VALUE" x="713.74" y="50.8" size="1.778" layer="96" rot="R90"/>
-</instance>
-<instance part="JP6" gate="A" x="767.08" y="96.52" smashed="yes">
-<attribute name="NAME" x="760.73" y="102.235" size="1.778" layer="95"/>
-<attribute name="VALUE" x="760.73" y="88.9" size="1.778" layer="96"/>
 </instance>
 </instances>
@@
 </segment>
 <segment>
+<pinref part="GND4" gate="1" pin="GND"/>
+<pinref part="JP4" gate="A" pin="3"/>
+<wire x1="810.26" y1="88.9" x2="800.1" y2="88.9" width="0.1524" layer="91"/>
+<pinref part="JP4" gate="A" pin="2"/>
+<wire x1="800.1" y1="88.9" x2="800.1" y2="91.44" width="0.1524" layer="91"/>
+<junction x="800.1" y="88.9"/>
+<pinref part="JP4" gate="A" pin="1"/>
+<wire x1="800.1" y1="91.44" x2="800.1" y2="93.98" width="0.1524" layer="91"/>
+<junction x="800.1" y="91.44"/>
+</segment>
+<segment>
 <pinref part="SW2" gate="G$1" pin="1"/>
 <pinref part="SW2" gate="G$1" pin="4"/>
@@
 <junction x="421.64" y="81.28"/>
 <pinref part="GND10" gate="1" pin="GND"/>
-</segment>
-<segment>
-<pinref part="JP6" gate="A" pin="1"/>
-<pinref part="JP6" gate="A" pin="3"/>
-<wire x1="764.54" y1="99.06" x2="764.54" y2="96.52" width="0.1524" layer="91"/>
-<pinref part="JP6" gate="A" pin="5"/>
-<wire x1="764.54" y1="96.52" x2="764.54" y2="93.98" width="0.1524" layer="91"/>
-<junction x="764.54" y="96.52"/>
-<pinref part="GND4" gate="1" pin="GND"/>
-<wire x1="764.54" y1="93.98" x2="764.54" y2="88.9" width="0.1524" layer="91"/>
-<junction x="764.54" y="93.98"/>
 </segment>
 </net>
@@
 </segment>
 <segment>
+<pinref part="JP3" gate="A" pin="1"/>
+<pinref part="JP3" gate="A" pin="2"/>
+<wire x1="800.1" y1="111.76" x2="800.1" y2="109.22" width="0.1524" layer="91"/>
+<pinref part="JP3" gate="A" pin="3"/>
+<wire x1="800.1" y1="109.22" x2="800.1" y2="106.68" width="0.1524" layer="91"/>
+<junction x="800.1" y="109.22"/>
+<pinref part="+3V6" gate="G$1" pin="+3V3"/>
+<wire x1="800.1" y1="111.76" x2="812.8" y2="111.76" width="0.1524" layer="91"/>
+<junction x="800.1" y="111.76"/>
+</segment>
+<segment>
 <pinref part="R5" gate="G$1" pin="2"/>
 <pinref part="+3V7" gate="G$1" pin="+3V3"/>
@@
 <pinref part="+3V15" gate="G$1" pin="+3V3"/>
 </segment>
-<segment>
-<pinref part="+3V6" gate="G$1" pin="+3V3"/>
-<pinref part="JP6" gate="A" pin="2"/>
-<wire x1="772.16" y1="109.22" x2="772.16" y2="99.06" width="0.1524" layer="91"/>
-<pinref part="JP6" gate="A" pin="4"/>
-<wire x1="772.16" y1="99.06" x2="772.16" y2="96.52" width="0.1524" layer="91"/>
-<junction x="772.16" y="99.06"/>
-<pinref part="JP6" gate="A" pin="6"/>
-<wire x1="772.16" y1="96.52" x2="772.16" y2="93.98" width="0.1524" layer="91"/>
-<junction x="772.16" y="96.52"/>
-</segment>
 </net>
