File: pcb/pboard_ibm_pc/rev1/ibmpc.brd (EAGLE design)
At the start: 56 x 65 mm, 48 parts, among them IC1 STM32F072C8T6, SW1 324_SW, SW2 324_SW, U1 MAX3232

Commit message: updated PCBs
Parts:
- added TP1, TP2: TPTP12R, testpad:TP12R
- added U$4: PINHD1X2, adafruit_changed:1X02
- moved R2 1.78 mm to (8.38, 27.9)
- moved R1 1.78 mm to (8.38, 30.0)
- moved C2 0.18 mm to (34.4, 36.0), turned to 0 degrees
Connections:
- new net N$3: J3.4_5V, U$8.1
- new net N$42: IC1.29, TP1.TP
- net +3V3: now also C6.2, R1.1, R2.1, R3.1, U$5.17
- net +5V: no longer C6.2, R1.1, R2.1, R3.1, U$5.17
- net N$4: no longer IC1.29
- net N$43: now also TP2.TP; no longer J3.4_5V, U$8.1
- net POT_SCL: now also U$4.2
- net PST_SDA: now also U$4.1
Routing:
- net +5V: track 157.3 -> 116.5 mm, vias 4 -> 2
- net N$43: track 36.6 -> 4.43 mm
- net +3V3: track 33.2 -> 48.9 mm, vias 6 -> 7
- net N$4: track 23.5 -> 8.38 mm, vias 1 -> 0
- net N$3: track 0.00 -> 8.59 mm
- net N$42: track 0.00 -> 3.85 mm, vias 0 -> 1
- net PST_SDA: track 24.5 -> 27.0 mm
- net POT_SCL: track 21.5 -> 23.4 mm
- net +UB: track 77.6 -> 78.5 mm
- net Y1_W0: track 19.0 -> 19.9 mm
Other:
- board text added: "A8"
- board text added: "B15"
- board text added: "SCL"
- board text added: "SDA"
