File: pcb/pboard_ibm_pc/rev1/ibmpc.sch (EAGLE design)
At the start: 48 parts, among them IC1 STM32F072C8T6, SW1 324_SW, SW2 324_SW, U1 MAX3232

Commit message: updated PCBs
Parts:
- added TP1, TP2: TPTP12R, testpad:TPTP12R
- added U$4: PINHD1X2, adafruit_changed:PINHD1X2
Connections:
- new net N$3: J3.4_5V, U$8.1
- new net N$42: IC1PORTA_H.PA8, TP1.TP
- net +3V3: now also C6.2, R1.1, R2.1, R3.1, U$5.VDD
- net +5V: no longer C6.2, R1.1, R2.1, R3.1, U$5.VDD
- net N$4: no longer IC1PORTA_H.PA8
- net N$43: now also TP2.TP; no longer J3.4_5V, U$8.1
- net POT_SCL: now also U$4.2
- net PST_SDA: now also U$4.1
