File: pcb/pboard_apple_all/apple_all.brd (EAGLE design)
At the start: 56 x 65 mm, 33 parts, among them IC1 STM32F072C8T6, SW1 324_SW, SW2 324_SW

Commit message: started quad encoder test
Parts:
- J2: device SparkFun-Connectors:DB9_MALE -> SparkFun-Connectors:DB9
Connections:
- new net +7V: J2.2
- new net MOUSE_BUTTON: J2.7
- new net X1: J2.5
- new net X2: J2.4
- new net Y1: J2.9
- new net Y2: J2.8
- net GND: now also J2.1, J2.3, J2.G1, J2.G2
Changed lines of the file:
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@@
 <attribute name="VALUE" x="-0.945" y="7.1" size="1.27" layer="28" rot="MR90"/>
 </element>
-<element name="J2" library="SparkFun-Connectors" package="DB9_MALE" value="" x="46.5" y="29" smashed="yes" rot="R270">
-<attribute name="PROD_ID" value="CONN-09904" x="46.5" y="29" size="1.778" layer="27" rot="R270" display="off"/>
+<element name="J2" library="SparkFun-Connectors" package="DB9" value="" x="46.5" y="29" smashed="yes" rot="R270">
+<attribute name="PROD_ID" value="CONN-08194" x="46.5" y="29" size="1.778" layer="27" rot="R270" display="off"/>
 <attribute name="VALUE" x="51.072" y="30.905" size="0.6096" layer="27" font="vector" ratio="20" rot="R270"/>
 </element>
@@
 <contactref element="U$8" pad="1"/>
 <contactref element="U$1" pad="1"/>
+<contactref element="J2" pad="1"/>
+<contactref element="J2" pad="3"/>
+<contactref element="J2" pad="G1"/>
+<contactref element="J2" pad="G2"/>
 <wire x1="36.83" y1="42.164" x2="28.829" y2="43.7752" width="0" layer="19" extent="1-1"/>
 </signal>
@@
 <wire x1="19.07" y1="50.5748" x2="21.2" y2="57.2" width="0" layer="19" extent="1-1"/>
 </signal>
+<signal name="+7V">
+<contactref element="J2" pad="2"/>
+</signal>
+<signal name="X2">
+<contactref element="J2" pad="4"/>
+</signal>
+<signal name="X1">
+<contactref element="J2" pad="5"/>
+</signal>
+<signal name="MOUSE_BUTTON">
+<contactref element="J2" pad="7"/>
+</signal>
+<signal name="Y2">
+<contactref element="J2" pad="8"/>
+</signal>
+<signal name="Y1">
+<contactref element="J2" pad="9"/>
+</signal>
 </signals>

Commit message: working on testing board
Parts:
- removed C6: 100nF, clock:0805@1
- added JP4, JP5: (no value), pinhead:2X04
- added JP6: (no value), pinhead:2X05
- added JP7: (no value), pinhead:1X05
- added JP8: (no value), pinhead:1X02
- added JP9: (no value), pinhead:1X04
- added R1, R10, R16, R17, R18, R19, R2, R20, R3, R4, R5, R6, R8: 5.1K, SparkFun-Passives:0805
- added SW3: 324_SW, 3pos_slide_switch_centered:342_SWICH_FOOT
- added U$11: RJ9PTH, SparkFun-Retired:RJ9
- moved LED1 42.0 mm to (11.2, 3.81)
- moved R7 42.0 mm to (8.64, 3.86)
- moved TP3 22.8 mm to (7.87, 56.0)
- moved U$9 11.4 mm to (19.8, 2.54)
- moved C7 2.68 mm to (24.7, 31.7), turned to 90 degrees
Connections:
- removed net +7V: J2.2
- removed net MOUSE_BUTTON: J2.7
- removed net N$44: IC1.20
- removed net X1: J2.5
- removed net X2: J2.4
- removed net Y1: J2.9
- removed net Y2: J2.8
- new net KB_5V: IC1.20, JP4.7, JP4.8, JP5.1, JP5.2, JP9.4, R16.1, R17.1, R18.1, R19.1, R20.1, R6.1
- new net KB_CLK: IC1.18, JP4.3, JP4.4, JP5.5, JP5.6, JP9.2, R19.2, R20.2, U$11.3, U$9.2
- new net KB_DATA: IC1.19, JP4.5, JP4.6, JP5.3, JP5.4, JP9.3, R17.2, R18.2, U$11.2, U$9.3
- new net N$26: J2.1, JP6.1
- new net N$30: J2.2, JP6.3
- new net N$31: J2.3, JP6.5
- new net N$32: J2.4, JP6.7
- new net N$33: J2.5, JP6.9
- new net N$34: J2.6, JP6.2
- new net N$35: J2.7, JP6.4
- new net N$36: J2.8, JP6.6
- new net N$42: J2.9, JP6.8
- new net N$43: IC1.45, U$1.3, U$4.ADB, U$5.ADB, U$8.3
- new net N$46: IC1.41, SW3.P$2, SW3.P$3, U$1.2, U$4.PSW, U$5.PSW, U$8.2
- new net N$47: IC1.25, JP7.5, R1.2
- new net N$48: IC1.29, JP7.1, R5.2
- new net N$49: JP8.1, JP8.2, R1.1, R2.1, R3.1, R4.1, R5.1
- new net N$5: R8.2, U$11.4
- new net N$50: R6.2, U$11.1
- new net N$51: R16.2, U$9.4
- new net N$52: R10.2, U$9.1
- net +3V3: now also JP3.5; no longer JP3.6
- net +5V: no longer C6.2
- net GND: now also JP3.6, JP4.1, JP4.2, JP5.7, JP5.8, JP6.10, JP9.1, R10.1, R8.1, SW3.P$1, SW3.P$4; no longer C6.1, J2.1, J2.3, JP3.5
- net N$10: now also IC1.27, JP7.3, R3.2; no longer U$1.2, U$4.PSW, U$5.PSW, U$8.2
- net N$3: now also IC1.46
- net N$4: now also IC1.28, JP7.2, R4.2; no longer U$1.3, U$4.ADB, U$5.ADB, U$8.3
- net N$45: now also IC1.26, JP7.4, R2.2; no longer IC1.18, TP3.TP
Routing:
- net N$46: track 0.00 -> 124.0 mm
- net KB_CLK: track 0.00 -> 61.8 mm
- net KB_DATA: track 0.00 -> 61.5 mm
- net KB_5V: track 0.00 -> 53.3 mm
- net N$43: track 0.00 -> 50.2 mm
- net N$3: track 0.00 -> 42.3 mm
- net N$48: track 0.00 -> 26.3 mm
- net N$4: track 0.00 -> 22.7 mm
- net N$10: track 0.00 -> 19.1 mm
- net N$45: track 0.00 -> 15.4 mm
- net N$49: track 0.00 -> 15.4 mm
- net +5V: track 125.9 -> 114.0 mm
- net N$26: track 0.00 -> 9.07 mm
- net N$32: track 0.00 -> 8.73 mm
- net N$33: track 0.00 -> 8.72 mm
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Other:
- board text added: "1"
- board text added: "2"
- board text added: "3"
- board text added: "4"
- board text added: "6"
- board text added: "7"
- board text added: "8"
- board text added: "9"
- board text added: "ADB PSW"
- board text added: "C"
- board text removed: "3V"
- board text removed: "B0"

Commit message: forgot what i did
Parts:
- added TP1, TP2: TPTP12R, testpad:TP12R
- moved TP3 22.3 mm to (24.0, 40.6)
Connections:
- new net N$11: IC1.40, TP3.TP
- new net N$17: IC1.21, TP1.TP
- new net N$19: IC1.22, TP2.TP
Routing:
- net N$11: track 0.00 -> 3.17 mm, vias 0 -> 1
- net N$17: track 0.00 -> 2.61 mm, vias 0 -> 1
- net N$19: track 0.00 -> 2.13 mm, vias 0 -> 1
Other:
- board text added: "A8"
- board text added: "B12"
- board text added: "B13"
- board text added: "B14"
- board text added: "B15"
- board text added: "PT1 dekuNukem APR2022"
- board text added: "USB4VC Protocol Card for Early Macintosh and Apple Desktop Bus"
- board text added: "git.io/usb4vc"
Changed lines of the file:
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@@
 <text x="19.05" y="24.638" size="1.143" layer="25" rot="R180" align="center">D</text>
 <text x="21.59" y="24.638" size="1.143" layer="25" rot="R180" align="center">5</text>
+<text x="28.2448" y="34.2646" size="1.143" layer="26" rot="MR180" align="center">B12</text>
+<text x="28.2448" y="31.7246" size="1.143" layer="26" rot="MR180" align="center">B13</text>
+<text x="28.2448" y="29.1846" size="1.143" layer="26" rot="MR180" align="center">B14</text>
+<text x="28.2448" y="26.6446" size="1.143" layer="26" rot="MR180" align="center">B15</text>
+<text x="28.3718" y="24.1046" size="1.143" layer="26" rot="MR180" align="center">A8</text>
+<text x="20.6248" y="43.9166" size="1.27" layer="26" rot="MR180" align="center">USB4VC Protocol Card for
+Early Macintosh
+and
+Apple Desktop Bus
+</text>
+<text x="21.1328" y="39.0906" size="1.27" layer="26" rot="MR180" align="center">PT1 dekuNukem APR2022</text>
+<text x="16.0528" y="31.3436" size="1.27" layer="26" rot="MR180" align="center">git.io/usb4vc</text>
 </plain>
 <attributes>
@@
 </element>
 <element name="U$10" library="adafruit_changed" package="1X04-CLEANBIG" value="PINHD1X4" x="12.954" y="34.29" smashed="yes"/>
-<element name="TP3" library="testpad" library_urn="urn:adsk.eagle:library:385" package="TP12R" package3d_urn="urn:adsk.eagle:package:27963/1" value="TPTP12R" x="7.874" y="56.007" smashed="yes" rot="MR0">
-<attribute name="POPULARITY" value="1" x="7.874" y="56.007" size="1.778" layer="28" rot="MR0" display="off"/>
-<attribute name="TP_SIGNAL_NAME" value="" x="7.874" y="56.007" size="1.778" layer="28" rot="MR0" display="off"/>
+<element name="TP3" library="testpad" library_urn="urn:adsk.eagle:library:385" package="TP12R" package3d_urn="urn:adsk.eagle:package:27963/1" value="TPTP12R" x="24.003" y="40.64" smashed="yes" rot="MR0">
+<attribute name="POPULARITY" value="1" x="24.003" y="40.64" size="1.778" layer="28" rot="MR0" display="off"/>
+<attribute name="TP_SIGNAL_NAME" value="" x="24.003" y="40.64" size="1.778" layer="28" rot="MR0" display="off"/>
 </element>
 <element name="JP2" library="pinhead" library_urn="urn:adsk.eagle:library:325" package="2X03" package3d_urn="urn:adsk.eagle:package:22462/2" value="" x="8.58" y="18.53" smashed="yes" rot="R90">
@@
 <element name="R20" library="SparkFun-Passives" package="0805" value="5.1K" x="19.05" y="21.59" smashed="yes" rot="R180">
 <attribute name="NAME" x="19.939" y="23.4315" size="0.8128" layer="25" rot="R180"/>
+</element>
+<element name="TP1" library="testpad" library_urn="urn:adsk.eagle:library:385" package="TP12R" package3d_urn="urn:adsk.eagle:package:27963/1" value="TPTP12R" x="21.971" y="36.576" smashed="yes" rot="MR0">
+<attribute name="POPULARITY" value="1" x="21.971" y="36.576" size="1.778" layer="28" rot="MR0" display="off"/>
+<attribute name="TP_SIGNAL_NAME" value="" x="21.971" y="36.576" size="1.778" layer="28" rot="MR0" display="off"/>
+</element>
+<element name="TP2" library="testpad" library_urn="urn:adsk.eagle:library:385" package="TP12R" package3d_urn="urn:adsk.eagle:package:27963/1" value="TPTP12R" x="23.622" y="36.576" smashed="yes" rot="MR0">
+<attribute name="POPULARITY" value="1" x="23.622" y="36.576" size="1.778" layer="28" rot="MR0" display="off"/>
+<attribute name="TP_SIGNAL_NAME" value="" x="23.622" y="36.576" size="1.778" layer="28" rot="MR0" display="off"/>
 </element>
 </elements>
@@
 <wire x1="53.086" y1="11.303" x2="48.26" y2="6.477" width="1.016" layer="16"/>
 <via x="46.101" y="49.911" extent="1-16" drill="0.55"/>
-<wire x1="53.086" y1="41.3766" x2="53.086" y2="11.303" width="1.016" layer="16"/>
-<wire x1="46.101" y1="48.3616" x2="53.086" y2="41.3766" width="1.016" layer="16"/>
-<wire x1="46.101" y1="48.3616" x2="46.101" y2="49.911" width="1.016" layer="16"/>
+<wire x1="53.086" y1="41.1226" x2="53.086" y2="11.303" width="1.016" layer="16"/>
+<wire x1="46.101" y1="48.1076" x2="53.086" y2="41.1226" width="1.016" layer="16"/>
+<wire x1="46.101" y1="48.1076" x2="46.101" y2="49.911" width="1.016" layer="16"/>
 <wire x1="46.101" y1="55.118" x2="46.101" y2="49.911" width="1.016" layer="16"/>
 <wire x1="48.2" y1="50.185" x2="46.375" y2="50.185" width="0.508" layer="1"/>
@@
 <contactref element="IC1" pad="14"/>
 <wire x1="19.75" y1="34.5" x2="19.75" y2="33.7962" width="0.1524" layer="1"/>
-<wire x1="19.75" y1="33.7962" x2="18.8468" y2="32.893" width="0.1524" layer="1"/>
-<wire x1="18.8468" y1="32.893" x2="8.5426" y2="32.893" width="0.1524" layer="1"/>
-<wire x1="8.5426" y1="32.893" x2="5.1256" y2="36.31" width="0.1524" layer="1"/>
-<wire x1="5.1256" y1="36.31" x2="4.77" y2="36.31" width="0.1524" layer="1"/>
+<wire x1="19.75" y1="33.7962" x2="18.7452" y2="32.7914" width="0.1524" layer="1"/>
+<wire x1="18.7452" y1="32.7914" x2="8.5172" y2="32.7914" width="0.1524" layer="1"/>
+<wire x1="8.5172" y1="32.7914" x2="4.9986" y2="36.31" width="0.1524" layer="1"/>
+<wire x1="4.9986" y1="36.31" x2="4.77" y2="36.31" width="0.1524" layer="1"/>
 </signal>
 <signal name="SPI_SCK">
@@
 <contactref element="JP1" pad="23"/>
 <wire x1="20.25" y1="34.5" x2="20.25" y2="33.712" width="0.1524" layer="1"/>
-<wire x1="20.25" y1="33.712" x2="18.9738" y2="32.4358" width="0.1524" layer="1"/>
-<wire x1="18.9738" y1="32.4358" x2="8.0772" y2="32.4358" width="0.1524" layer="1"/>
-<wire x1="8.0772" y1="32.4358" x2="5.4864" y2="35.0266" width="0.1524" layer="1"/>
+<wire x1="20.25" y1="33.712" x2="18.8214" y2="32.2834" width="0.1524" layer="1"/>
+<wire x1="18.8214" y1="32.2834" x2="8.2296" y2="32.2834" width="0.1524" layer="1"/>
+<wire x1="8.2296" y1="32.2834" x2="5.4864" y2="35.0266" width="0.1524" layer="1"/>
 <wire x1="5.4864" y1="35.0266" x2="3.5134" y2="35.0266" width="0.1524" layer="1"/>
 <wire x1="3.5134" y1="35.0266" x2="2.23" y2="36.31" width="0.1524" layer="1"/>
@@
 <contactref element="JP1" pad="21"/>
 <wire x1="20.75" y1="34.5" x2="20.75" y2="33.577" width="0.1524" layer="1"/>
-<wire x1="20.75" y1="33.577" x2="19.177" y2="32.004" width="0.1524" layer="1"/>
-<wire x1="19.177" y1="32.004" x2="5.969" y2="32.004" width="0.1524" layer="1"/>
-<wire x1="5.969" y1="32.004" x2="5.461" y2="32.512" width="0.1524" layer="1"/>
+<wire x1="20.75" y1="33.577" x2="18.9484" y2="31.7754" width="0.1524" layer="1"/>
+<wire x1="18.9484" y1="31.7754" x2="6.1976" y2="31.7754" width="0.1524" layer="1"/>
+<wire x1="6.1976" y1="31.7754" x2="5.461" y2="32.512" width="0.1524" layer="1"/>
 <wire x1="5.461" y1="32.512" x2="3.488" y2="32.512" width="0.1524" layer="1"/>
 <wire x1="3.488" y1="32.512" x2="2.23" y2="33.77" width="0.1524" layer="1"/>
@@
 <wire x1="21.25" y1="34.5" x2="21.25" y2="33.3658" width="0.1524" layer="1"/>
 <wire x1="5.4864" y1="29.9466" x2="3.5134" y2="29.9466" width="0.1524" layer="1"/>
-<wire x1="21.25" y1="33.3658" x2="19.431" y2="31.5468" width="0.1524" layer="1"/>
-<wire x1="19.431" y1="31.5468" x2="7.0866" y2="31.5468" width="0.1524" layer="1"/>
-<wire x1="7.0866" y1="31.5468" x2="5.4864" y2="29.9466" width="0.1524" layer="1"/>
+<wire x1="21.25" y1="33.3658" x2="19.177" y2="31.2928" width="0.1524" layer="1"/>
+<wire x1="19.177" y1="31.2928" x2="6.8326" y2="31.2928" width="0.1524" layer="1"/>
+<wire x1="6.8326" y1="31.2928" x2="5.4864" y2="29.9466" width="0.1524" layer="1"/>
 </signal>
 <signal name="N$1">
@@
 <wire x1="42.153" y1="11.43" x2="42.164" y2="11.419" width="0.2032" layer="1"/>
 </signal>
+<signal name="N$11">
+<contactref element="IC1" pad="40"/>
+<contactref element="TP3" pad="TP"/>
+<wire x1="23.25" y1="43.5" x2="23.25" y2="42.409" width="0.1524" layer="1"/>
+<wire x1="24.003" y1="41.656" x2="24.003" y2="40.64" width="0.1524" layer="1"/>
+<via x="24.003" y="40.64" extent="1-16" drill="0.5"/>
+<wire x1="23.25" y1="42.409" x2="24.003" y2="41.656" width="0.1524" layer="1"/>
+</signal>
+<signal name="N$17">
+<contactref element="IC1" pad="21"/>
+<contactref element="TP1" pad="TP"/>
+<wire x1="23.25" y1="34.5" x2="23.25" y2="35.297" width="0.1524" layer="1"/>
+<via x="21.971" y="36.576" extent="1-16" drill="0.5"/>
+<wire x1="23.25" y1="35.297" x2="21.971" y2="36.576" width="0.1524" layer="1"/>
+</signal>
+<signal name="N$19">
+<contactref element="IC1" pad="22"/>
+<contactref element="TP2" pad="TP"/>
+<wire x1="23.75" y1="34.5" x2="23.75" y2="36.448" width="0.1524" layer="1"/>
+<wire x1="23.75" y1="36.448" x2="23.622" y2="36.576" width="0.1524" layer="1"/>
+<via x="23.622" y="36.576" extent="1-16" drill="0.5"/>
+</signal>
 </signals>
 <mfgpreviewcolors>
@@
 <mfgpreviewcolor name="substratecolor" color="0xFF786E46"/>
 </mfgpreviewcolors>
+<errors>
+</errors>
 </board>
 </drawing>
 <compatibility>
+<note version="6.3" minversion="6.2.2" severity="warning">
+Since Version 6.2.2 text objects can contain more than one line,
+which will not be processed correctly with this version.
+</note>
 <note version="8.2" severity="warning">
 Since Version 8.2, EAGLE supports online libraries. The ids
