File: pcb/pboard_apple_all/apple_all_pt3.brd (EAGLE design)
At the start: 56 x 65 mm, 47 parts, among them IC1 STM32F072C8T6, SW1 324_SW, SW2 324_SW, SW3 324_SW

Commit message: adjusted prototype pcb
Parts:
- moved R8 5.04 mm to (30.0, 22.0)
- moved R10 5.04 mm to (31.9, 22.0)
- moved R16 5.04 mm to (28.1, 22.0)
- moved R6 5.04 mm to (33.9, 22.0)
- moved U$9 3.86 mm to (35.6, 6.59)
Routing:
- net N$30: track 12.5 -> 17.1 mm
- net N$25: track 12.3 -> 16.9 mm
- net N$17: track 12.9 -> 17.4 mm
- net N$19: track 12.2 -> 16.6 mm
- net N$21: track 12.8 -> 10.5 mm
- net N$10: track 13.5 -> 11.1 mm
- net N$20: track 9.20 -> 7.22 mm
- net N$5: track 9.12 -> 7.21 mm
- net N$4: track 43.6 -> 44.3 mm
