File: pcb/bbc_micro/bbc_micro.sch (EAGLE design)
At the start: 27 parts, among them IC1 STM32F072C8T6, SW1 324_SW, SW2 324_SW, SW3 324_SW

Commit message: working on bbc micro PCB
Parts:
- added U$9: GAMEPORT_15P, ibmpc:GAMEPORT_15P
- JP3: device pinhead:PINHD-2X4 -> pinhead:PINHD-2X3
Connections:
- removed net N$27: IC1PORTA_H.PA15, JP3.1, R15.1
- removed net N$6: IC1PORTB_L.PB3, JP3.2, R12.1
- net +3V3: now also JP3.3; no longer JP3.5
- net GND: now also JP3.4; no longer JP3.6
- net N$12: now also JP3.5; no longer JP3.7
- net N$14: now also JP3.6; no longer JP3.8
- net N$15: now also JP3.1; no longer JP3.3
- net N$16: now also JP3.2; no longer JP3.4
- net N$8: now also R12.1
- net N$9: now also R15.1
Other:
- note added: "PIN 1"
- moved on the sheet: IC1PORTB_H, LED2, LED3, R12, R15

Commit message: almost done with pcb
Parts:
- added C1: 100nF, clock:CAP0805
- added R1, R16, R17, R18, R19, R2, R3, R4, R5, R6, R8: 5.1K, SparkFun-Passives:RESISTOR0805-RES
- added R10: 2K, SparkFun-Passives:RESISTOR0805-RES
- added U$5: MCP4451, ps2:MCP4451
- U$9: value GAMEPORT_15P -> BBC_15P; device ibmpc:GAMEPORT_15P -> bbc_micro:BBC_15P
Connections:
- new net N$10: U$5.P2W, U$9.12_CH2
- new net N$11: U$5.P0W, U$9.4_CH3
- new net N$17: U$5.P1A, U$5.P3B, U$9.14_VREF
- new net N$19: U$5.P0A, U$5.P2B, U$9.11_VREF
- new net N$20: R18.1, R19.1, U$9.1_5V
- new net N$21: R18.2, U$9.10_PB1
- new net N$24: R19.2, U$9.13_PB0
- new net N$4: R10.1, U$5.HVC/A0
- new net N$5: U$5.P3W, U$9.7_CH1
- new net N$6: U$5.P1W, U$9.15_CH0
- net +3V3: now also C1.2, R16.2, R17.2, U$5.VDD
- net /EN: now also IC1PORTB_L.PB2
- net BREAK: now also IC1PORTB_L.PB1
- net CA2: now also IC1PORTB_H.PB15
- net CB1/XA: now also IC1PORTC.PC15, R1.1
- net CB2/YA: now also IC1PORTC.PC14, R2.1
- net D0/XD: now also IC1PORTC.PC13, R3.1
- net D2/YD: now also IC1PORTB_L.PB5, R4.1
- net D5/LEFT: now also IC1PORTB_L.PB4, R5.1
- net D6/MIDDLE: now also IC1PORTB_L.PB3, R6.1
- net D7/RIGHTT: now also IC1PORTA_H.PA15, R8.1
- net GND: now also C1.1, R10.2, U$5.A1, U$5.VSS, U$9.2_0V, U$9.3_0V, U$9.5_AGND, U$9.6_0V, U$9.8_AGND
- net N$22: now also R16.1, U$5.SCL
- net N$23: now also R17.1, U$5.SDA
- net N$37: now also IC1PORTF/OSC.PF1/OSC=>; no longer IC1PORTC.PC13
- net USER_PORT_5V: now also R1.2, R2.2, R3.2, R4.2, R5.2, R6.2, R8.2
- net W: now also IC1PORTA_H.PA8
Other:
- moved on the sheet: C7, C8, C9, IC1PORTB_H, IC1PORTC, IC1PORTF/OSC, JP2, JP4

Commit message: hooked up digital pot and leds
Parts:
- added LED4, LED5, LED6: (no value), adafruit:LEDCHIP-LED0805
- added R20: 5.1K, SparkFun-Passives:RESISTOR0805-RES
- added R21, R22, R23: 2K, SparkFun-Passives:RESISTOR0805-RES
Connections:
- removed net N$24: R19.2, U$9.13_PB0
- new net N$25: IC1PORTB_L.PB0, R20.1, U$5./RESET
- new net N$26: LED5.C, R22.2
- new net N$27: LED6.C, R23.2
- new net N$30: IC1PORTA_L.PA2, R19.2, U$9.13_PB0
- net BREAK: now also SW3.2, SW3.3
- net GND: now also R20.2
- net KB_5V: now also R21.1, R22.1, R23.1
- net LED_CAPSLOCK: now also LED6.A
- net LED_CASSETTE: now also LED4.A
- net LED_SHIFTLOCK: now also LED5.A
- net N$21: now also IC1PORTA_L.PA3
- net N$3: now also LED4.C, R21.2; no longer SW3.2, SW3.3

Commit message: bbc micro protocol board test board
Parts:
- added U$1: PINHD1X2, adafruit_changed:PINHD1X2
Connections:
- new net N$24: IC1PORTA_L.PA0, U$1.1
- new net N$31: IC1PORTA_L.PA1, U$1.2
Changed lines of the file:
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@@
 <part name="LED6" library="adafruit" deviceset="LED" device="CHIP-LED0805"/>
 <part name="R23" library="SparkFun-Passives" deviceset="RESISTOR" device="0805-RES" value="2K"/>
+<part name="U$1" library="adafruit_changed" deviceset="PINHD1X2" device=""/>
 </parts>
 <sheets>
@@
 <attribute name="NAME" x="288.29" y="-82.7786" size="1.778" layer="95" rot="R180"/>
 <attribute name="VALUE" x="288.29" y="-77.978" size="1.778" layer="96" rot="R180"/>
+</instance>
+<instance part="U$1" gate="1" x="53.34" y="25.4" smashed="yes">
+<attribute name="NAME" x="46.99" y="31.115" size="1.778" layer="95"/>
+<attribute name="VALUE" x="46.99" y="20.32" size="1.778" layer="96"/>
 </instance>
 </instances>
@@
 </segment>
 </net>
+<net name="N$24" class="0">
+<segment>
+<pinref part="IC1" gate="PORTA_L" pin="PA0"/>
+<pinref part="U$1" gate="1" pin="1"/>
+<wire x1="43.18" y1="27.94" x2="50.8" y2="27.94" width="0.1524" layer="91"/>
+</segment>
+</net>
+<net name="N$31" class="0">
+<segment>
+<pinref part="U$1" gate="1" pin="2"/>
+<pinref part="IC1" gate="PORTA_L" pin="PA1"/>
+<wire x1="50.8" y1="25.4" x2="43.18" y2="25.4" width="0.1524" layer="91"/>
+</segment>
+</net>
