File: pcb/bbc_micro/pt0/bbc_micro.brd (EAGLE design)
At the start: 56 x 65 mm, 52 parts, among them IC1 STM32F072C8T6, SW1 324_SW, SW2 324_SW, SW3 324_SW

Commit message: updated bbc pcard
Parts:
- removed R24, R25: 2K, SparkFun-Passives:0805
Connections:
- net CA2: no longer R25.1
- net KB_5V: no longer R24.2, R25.2
- net W: no longer R24.1
Changed lines of the file:
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@@
 </element>
 <element name="U$1" library="adafruit_changed" package="1X02" value="PINHD1X2" x="15.367" y="35.687" smashed="yes" rot="R270"/>
-<element name="R24" library="SparkFun-Passives" package="0805" value="2K" x="-1.524" y="-4.445" smashed="yes">
-<attribute name="NAME" x="-2.286" y="-3.6195" size="0.8128" layer="25"/>
-</element>
-<element name="R25" library="SparkFun-Passives" package="0805" value="2K" x="-4.572" y="-4.445" smashed="yes">
-<attribute name="NAME" x="-5.334" y="-3.6195" size="0.8128" layer="25"/>
-</element>
 </elements>
 <signals>
@@
 <wire x1="37.742" y1="38.25" x2="41.612" y2="42.12" width="0.2032" layer="1"/>
 <wire x1="42.418" y1="42.12" x2="44.958" y2="42.12" width="0.2032" layer="16"/>
-<contactref element="R24" pad="1"/>
-<wire x1="-2.424" y1="-4.445" x2="26.5" y2="38.25" width="0" layer="19" extent="1-1"/>
 </signal>
 <signal name="LED_CASSETTE">
@@
 <wire x1="43.307" y1="40.894" x2="43.7134" y2="41.3004" width="0.2032" layer="1"/>
 <wire x1="42.418" y1="47.2" x2="44.958" y2="47.2" width="0.2032" layer="16"/>
-<contactref element="R25" pad="1"/>
-<wire x1="-5.472" y1="-4.445" x2="26.5" y2="37.75" width="0" layer="19" extent="1-1"/>
 </signal>
 <signal name="KB_5V">
@@
 <wire x1="33.528" y1="29.718" x2="30.723" y2="29.718" width="0.2032" layer="1"/>
 <wire x1="42.418" y1="49.74" x2="44.958" y2="49.74" width="0.2032" layer="16"/>
-<contactref element="R24" pad="2"/>
-<contactref element="R25" pad="2"/>
-<wire x1="-0.624" y1="-4.445" x2="30.723" y2="28.321" width="0" layer="19" extent="1-1"/>
-<wire x1="-3.672" y1="-4.445" x2="-0.624" y2="-4.445" width="0" layer="19" extent="1-1"/>
 </signal>
 <signal name="LED_SHIFTLOCK">
