File: pcb/bbc_micro/pt0/bbc_micro.sch (EAGLE design)
At the start: 52 parts, among them IC1 STM32F072C8T6, SW1 324_SW, SW2 324_SW, SW3 324_SW

Commit message: updated bbc pcard
Parts:
- removed R24, R25: 2K, SparkFun-Passives:RESISTOR0805-RES
Connections:
- net CA2: no longer R25.1
- net KB_5V: no longer R24.2, R25.2
- net W: no longer R24.1
Changed lines of the file:
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@@
 <part name="R23" library="SparkFun-Passives" deviceset="RESISTOR" device="0805-RES" value="2K"/>
 <part name="U$1" library="adafruit_changed" deviceset="PINHD1X2" device=""/>
-<part name="R24" library="SparkFun-Passives" deviceset="RESISTOR" device="0805-RES" value="2K"/>
-<part name="R25" library="SparkFun-Passives" deviceset="RESISTOR" device="0805-RES" value="2K"/>
 </parts>
 <sheets>
@@
 <attribute name="VALUE" x="-76.2" y="-53.34" size="1.778" layer="96" rot="R90"/>
 </instance>
-<instance part="SW3" gate="G$1" x="309.88" y="-17.78" smashed="yes" rot="MR270"/>
-<instance part="GND13" gate="1" x="312.42" y="-38.1" smashed="yes">
-<attribute name="VALUE" x="309.88" y="-40.64" size="1.778" layer="96"/>
+<instance part="SW3" gate="G$1" x="281.94" y="-17.78" smashed="yes" rot="MR270"/>
+<instance part="GND13" gate="1" x="284.48" y="-38.1" smashed="yes">
+<attribute name="VALUE" x="281.94" y="-40.64" size="1.778" layer="96"/>
 </instance>
 <instance part="JP7" gate="A" x="-58.42" y="-48.26" smashed="yes">
@@
 <attribute name="NAME" x="46.99" y="31.115" size="1.778" layer="95"/>
 <attribute name="VALUE" x="46.99" y="20.32" size="1.778" layer="96"/>
-</instance>
-<instance part="R24" gate="G$1" x="287.02" y="-33.02" smashed="yes" rot="R270">
-<attribute name="NAME" x="288.5186" y="-29.21" size="1.778" layer="95" rot="R270"/>
-<attribute name="VALUE" x="283.718" y="-29.21" size="1.778" layer="96" rot="R270"/>
-</instance>
-<instance part="R25" gate="G$1" x="279.4" y="-38.1" smashed="yes" rot="R270">
-<attribute name="NAME" x="280.8986" y="-34.29" size="1.778" layer="95" rot="R270"/>
-<attribute name="VALUE" x="276.098" y="-34.29" size="1.778" layer="96" rot="R270"/>
 </instance>
 </instances>
@@
 <pinref part="SW3" gate="G$1" pin="1"/>
 <pinref part="SW3" gate="G$1" pin="4"/>
-<wire x1="312.42" y1="-2.54" x2="312.42" y2="-33.02" width="0.1524" layer="91"/>
+<wire x1="284.48" y1="-2.54" x2="284.48" y2="-33.02" width="0.1524" layer="91"/>
 <pinref part="GND13" gate="1" pin="GND"/>
-<wire x1="312.42" y1="-35.56" x2="312.42" y2="-33.02" width="0.1524" layer="91"/>
-<junction x="312.42" y="-33.02"/>
+<wire x1="284.48" y1="-35.56" x2="284.48" y2="-33.02" width="0.1524" layer="91"/>
+<junction x="284.48" y="-33.02"/>
 </segment>
 <segment>
@@
 <pinref part="SW3" gate="G$1" pin="3"/>
 <pinref part="SW3" gate="G$1" pin="2"/>
-<wire x1="304.8" y1="-2.54" x2="304.8" y2="-33.02" width="0.1524" layer="91"/>
-<wire x1="254" y1="-2.54" x2="304.8" y2="-2.54" width="0.1524" layer="91"/>
+<wire x1="276.86" y1="-2.54" x2="276.86" y2="-33.02" width="0.1524" layer="91"/>
+<wire x1="254" y1="-2.54" x2="276.86" y2="-2.54" width="0.1524" layer="91"/>
 <junction x="254" y="-2.54"/>
-<junction x="304.8" y="-2.54"/>
+<junction x="276.86" y="-2.54"/>
 </segment>
 </net>
@@
 <junction x="246.38" y="-27.94"/>
 <pinref part="IC1" gate="PORTA_H" pin="PA8"/>
-<wire x1="40.64" y1="-38.1" x2="182.88" y2="-38.1" width="0.1524" layer="91"/>
+<wire x1="40.64" y1="-38.1" x2="144.78" y2="-38.1" width="0.1524" layer="91"/>
+<wire x1="149.86" y1="-38.1" x2="144.78" y2="-38.1" width="0.1524" layer="91"/>
+<wire x1="149.86" y1="-38.1" x2="182.88" y2="-38.1" width="0.1524" layer="91"/>
 <wire x1="182.88" y1="-38.1" x2="182.88" y2="-27.94" width="0.1524" layer="91"/>
-<pinref part="R24" gate="G$1" pin="1"/>
-<wire x1="254" y1="-27.94" x2="287.02" y2="-27.94" width="0.1524" layer="91"/>
-<junction x="254" y="-27.94"/>
 </segment>
 </net>
@@
 <pinref part="IC1" gate="PORTB_H" pin="PB15"/>
 <wire x1="167.64" y1="-27.94" x2="167.64" y2="-33.02" width="0.1524" layer="91"/>
-<pinref part="R25" gate="G$1" pin="1"/>
-<wire x1="254" y1="-33.02" x2="279.4" y2="-33.02" width="0.1524" layer="91"/>
-<junction x="254" y="-33.02"/>
 </segment>
 </net>
@@
 <junction x="254" y="-35.56"/>
 <wire x1="274.32" y1="-35.56" x2="274.32" y2="-53.34" width="0.1524" layer="91"/>
-<wire x1="274.32" y1="-53.34" x2="279.4" y2="-53.34" width="0.1524" layer="91"/>
+<wire x1="274.32" y1="-53.34" x2="289.56" y2="-53.34" width="0.1524" layer="91"/>
 <pinref part="R21" gate="G$1" pin="1"/>
-<wire x1="279.4" y1="-53.34" x2="287.02" y2="-53.34" width="0.1524" layer="91"/>
-<wire x1="287.02" y1="-53.34" x2="289.56" y2="-53.34" width="0.1524" layer="91"/>
 <wire x1="289.56" y1="-53.34" x2="289.56" y2="-60.96" width="0.1524" layer="91"/>
 <pinref part="R22" gate="G$1" pin="1"/>
@@
 <wire x1="289.56" y1="-71.12" x2="289.56" y2="-81.28" width="0.1524" layer="91"/>
 <junction x="289.56" y="-71.12"/>
-<pinref part="R24" gate="G$1" pin="2"/>
-<wire x1="287.02" y1="-38.1" x2="287.02" y2="-53.34" width="0.1524" layer="91"/>
-<junction x="287.02" y="-53.34"/>
-<pinref part="R25" gate="G$1" pin="2"/>
-<wire x1="279.4" y1="-43.18" x2="279.4" y2="-53.34" width="0.1524" layer="91"/>
-<junction x="279.4" y="-53.34"/>
-</segment>
-</net>
+</segment>
+</net>
