File: pcb/bbc_micro/pt1/bbc_micro.sch (EAGLE design)
At the start: 51 parts, among them IC1 STM32F072C8T6, SW1 324_SW, SW2 324_SW, SW3 324_SW

Commit message: changed to using built-in DAC
Parts:
- removed JP5: (no value), pinhead:PINHD-1X2
- removed R26: 5.1K, SparkFun-Passives:RESISTOR0805-RES
- added C1: 100nF, clock:CAP0805
- added U$1: PINHD1X2, adafruit_changed:PINHD1X2
- added U$5: MCP4451, ps2:MCP4451
- R10: value 5.1K -> 2K
Connections:
- removed net N$12 (its old number): IC1PORTB_L.PB0, R17.2, R20.1, U$9.4_CH3
- new net N$10: U$5.P2W, U$9.12_CH2
- new net N$19: U$5.P0A, U$5.P2B, U$9.11_VREF
- new net N$24: IC1PORTA_L.PA0, U$1.1
- new net N$25: IC1PORTB_L.PB0, R20.1, U$5./RESET
- new net N$31: IC1PORTA_L.PA1, U$1.2
- new net N$6: U$5.P1W, U$9.15_CH0
- net +3V3: now also C1.2, IC1AN_POWER.VDDA, R16.2, R17.2, U$5.VDD
- net BREAK: no longer JP5.1
- net CLK: no longer R26.1
- net D6/MIDDLE: now also IC1PORTB_L.PB3; no longer IC1PORTF/OSC.PF0/OSC<=
- net D7/RIGHTT: now also IC1PORTA_H.PA15; no longer IC1PORTA_L.PA0
- net GND: now also C1.1, R10.2, U$5.A1, U$5.VSS; no longer JP5.2, R16.2, R26.2
- net N$11: now also U$5.P0W, U$9.4_CH3; no longer IC1AN_POWER.VDDA, R10.1, R17.1, U$9.11_VREF, U$9.14_VREF
- net N$17: now also U$5.P1A, U$5.P3B, U$9.14_VREF; no longer IC1PORTA_L.PA1, R10.2, R16.1, U$9.12_CH2
- net N$22: now also R16.1, U$5.SCL
- net N$23: now also R17.1, U$5.SDA
- net N$4: now also R10.1, U$5.HVC/A0; no longer IC1PORTA_L.PA4, U$9.15_CH0
- net N$5: now also U$5.P3W; no longer IC1PORTA_L.PA5
- net SPI_CS: now also IC1PORTA_L.PA4; no longer IC1PORTA_H.PA15
- net SPI_SCK: now also IC1PORTA_L.PA5; no longer IC1PORTB_L.PB3
Other:
- moved on the sheet: R10, R16, R17, R20
