File: pcb/sirius1_victor9000/sirius1.brd (EAGLE design)
At the start: 56 x 65 mm, 33 parts, among them IC3 STM32F042F4, SW1 324_SW, SW4 324_SW, U1 RJ45

Commit message: forgot what i did
Connections:
- net GND: now also TP1.TP, TP2.TP
Changed lines of the file:
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@@
 <text x="12.8016" y="27.9908" size="1.143" layer="25" rot="R90" align="center">POWER</text>
 <text x="11.2776" y="36.3474" size="1.6764" layer="25" rot="R90" align="center">RST</text>
-<text x="24.0538" y="44.5262" size="1.143" layer="25" rot="R180" align="center">ACT</text>
+<text x="24.0538" y="47.9552" size="1.143" layer="25" rot="R180" align="center">ACT</text>
 <text x="48.133" y="50.165" size="1.143" layer="25" rot="R180" align="center">TX</text>
 <text x="11.3284" y="44.4246" size="1.6764" layer="25" rot="R270" align="center">DFU</text>
@@
 <contactref element="JP2" pad="4"/>
 <contactref element="JP2" pad="2"/>
+<contactref element="TP2" pad="TP"/>
+<contactref element="TP1" pad="TP"/>
 </signal>
 <signal name="+3V3">
