File: pcb/sirius1_victor9000/pt0/sirius1.brd (EAGLE design)
At the start: 56 x 65 mm, 28 parts, among them IC3 STM32F042F4, SW1 324_SW, SW4 324_SW, U1 RJ45

Commit message: updated sirius 1 pcb
Parts:
- added JP2, JP6: (no value), pinhead:2X04
- added JP8: (no value), pinhead:2X05
- added R11, R12: 5.1K, SparkFun-Passives:0805
- JP3: device pinhead:1X05 -> pinhead:2X04
- moved R10 17.5 mm to (37.8, 27.2), turned to 270 degrees
- moved R9 13.9 mm to (35.3, 27.2), turned to 270 degrees
- moved R8 10.3 mm to (32.8, 27.2), turned to 270 degrees
- moved JP3 3.14 mm to (26.7, 16.8), turned to 90 degrees
- moved R3 2.42 mm to (49.8, 28.4), turned to 180 degrees
Connections:
- removed net KBACK: IC3.14, JP3.4, R10.1, U1.4
- removed net KBDATA: IC3.6, JP3.2, R8.1, U1.6
- removed net KBRDY: IC3.9, JP3.3, R9.1, U1.5
- removed net N$3: IC3.17, J4.A7, J4.B7
- new net N$15: JP3.2, JP6.2, U1.2
- new net N$16: JP3.3, JP6.3, U1.3
- new net N$18: JP3.4, JP6.4, U1.4
- new net N$19: JP3.5, JP6.5, U1.5
- new net N$20: JP3.6, JP6.6, U1.6
- new net N$21: JP3.7, JP6.7, U1.7
- new net N$22: JP3.8, JP6.8, U1.8
- new net N$24: IC3.9, JP8.3, JP8.4, R9.1
- new net N$25: IC3.14, JP8.5, JP8.6, R10.1
- new net N$26: IC3.18, J4.A6, J4.B6, JP8.10, JP8.9, R12.1
- new net N$30: IC3.6, JP8.1, JP8.2, R8.1
- new net N$4: IC3.17, J4.A7, J4.B7, JP8.7, JP8.8, R11.1
- net GND: now also JP2.2, JP2.4, JP2.6, JP2.8; no longer JP3.5, U1.2, U1.3, U1.8
- net N$14: now also JP3.1, JP6.1, U1.1; no longer IC3.18, J4.A6, J4.B6
- net N$27: now also JP2.1, JP2.3, JP2.5, JP2.7, R11.2, R12.2; no longer JP3.1, U1.1, U1.7
Routing:
- net N$26: track 0.00 -> 46.6 mm
- net KBACK: track 42.9 -> 0.00 mm
- net KBRDY: track 40.3 -> 0.00 mm, vias 1 -> 0
- net KBDATA: track 34.7 -> 0.00 mm, vias 1 -> 0
- net N$4: track 0.00 -> 31.9 mm
- net N$3: track 22.2 -> 0.00 mm
- net N$22: track 0.00 -> 21.5 mm
- net N$18: track 0.00 -> 21.5 mm
- net N$15: track 0.00 -> 21.5 mm
- net N$20: track 0.00 -> 21.4 mm
- net N$21: track 0.00 -> 21.0 mm
- net N$19: track 0.00 -> 21.0 mm
- net N$16: track 0.00 -> 21.0 mm
- net N$27: track 41.8 -> 24.0 mm
- net N$30: track 0.00 -> 17.6 mm, vias 0 -> 1
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Other:
- board text added: "1"
- board text added: "2"
- board text added: "3"
- board text added: "4"
- board text added: "5"
- board text added: "6"
- board text added: "7"
- board text added: "8"
- board text added: "A0"
- board text added: "A10"
- board text added: "A3"
- board text added: "A9"
- board text added: "B1"
- board text added: "VCC"
- board text added: "usb4vc.com dekuNukem PT1 NOV 2022"
- board text removed: "ACK"
- board text removed: "DAT"
- board text removed: "KB5V"
- board text removed: "RDY"
- board text removed: "usb4vc.com dekuNukem PT2 NOV 2022"
