File: pcb/sirius1_victor9000_trs80_model_2/sirius1_trs80_model_2.brd (EAGLE design)
At the start: 56 x 65 mm, 30 parts, among them IC3 STM32F042F4, SW1 324_SW, SW4 324_SW, U1 RJ45

Commit message: adjusted footprint
Parts:
- TP1, TP2: value TPSQPAD1-20 -> TPSQPAD1-17; device testpad:P1-20 -> testpad:P1-17
- moved U$1 2.00 mm to (42.4, 39.9)
- moved U1 2.00 mm to (47.1, 16.5)
- moved TP1 0.82 mm to (50.5, 24.5)
- moved TP2 0.82 mm to (50.5, 8.56)
Routing:
- net KBACK: track 49.6 -> 57.6 mm
- net KBDATA: track 48.6 -> 52.6 mm
- net +5V: track 106.4 -> 109.7 mm
- net KBRDY: track 53.9 -> 57.1 mm
- net N$27: track 80.0 -> 82.2 mm
