File: pcb/sirius1_victor9000_trs80_model_2/sirius1_trs80_model_2.sch (EAGLE design)
At the start: 30 parts, among them IC3 STM32F042F4, SW1 324_SW, SW4 324_SW, U1 RJ45

Commit message: adjusted footprint
Parts:
- TP1, TP2: value TPSQPAD1-20 -> TPSQPAD1-17; device testpad:TPSQPAD1-20 -> testpad:TPSQPAD1-17
Changed lines of the file:
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@@
 <part name="R10" library="SparkFun-Passives" deviceset="RESISTOR" device="0805-RES" value="5.1K"/>
 <part name="GND10" library="supply1" library_urn="urn:adsk.eagle:library:371" deviceset="GND" device=""/>
-<part name="TP1" library="testpad" library_urn="urn:adsk.eagle:library:385" deviceset="TPSQ" device="PAD1-20" package3d_urn="urn:adsk.eagle:package:27950/1"/>
-<part name="TP2" library="testpad" library_urn="urn:adsk.eagle:library:385" deviceset="TPSQ" device="PAD1-20" package3d_urn="urn:adsk.eagle:package:27950/1"/>
+<part name="TP1" library="testpad" library_urn="urn:adsk.eagle:library:385" deviceset="TPSQ" device="PAD1-17" package3d_urn="urn:adsk.eagle:package:27949/1" value="TPSQPAD1-17"/>
+<part name="TP2" library="testpad" library_urn="urn:adsk.eagle:library:385" deviceset="TPSQ" device="PAD1-17" package3d_urn="urn:adsk.eagle:package:27949/1" value="TPSQPAD1-17"/>
 <part name="GND11" library="supply1" library_urn="urn:adsk.eagle:library:371" deviceset="GND" device=""/>
 <part name="GND13" library="supply1" library_urn="urn:adsk.eagle:library:371" deviceset="GND" device=""/>
